Commit message: ros2 control via thunder_ahand_library

File: src/allegro_hand_description/urdf/allegro_hand_description_right_B.urdf (robot description, URDF)
Before this commit: robot allegro_hand_right, 22 links, 21 joints
Links:
- link link_0_0: geometry collision mesh filename=package://allegro_hand_description/meshes/new_l1.stl scale=0.001 0.001 0.001; visual mesh filename=package://allegro_hand_description/meshes/new_l1.stl scale=0.001 0.001 0.001
- link link_10_0: geometry collision mesh filename=package://allegro_hand_description/meshes/new_l3.stl scale=0.001 0.001 0.001; visual mesh filename=package://allegro_hand_description/meshes/new_l3.stl scale=0.001 0.001 0.001
- link link_11_0: geometry collision mesh filename=package://allegro_hand_description/meshes/new_l4.stl scale=0.001 0.001 0.001; visual mesh filename=package://allegro_hand_description/meshes/new_l4.stl scale=0.001 0.001 0.001
- link link_11_0_tip: geometry collision mesh filename=package://allegro_hand_description/meshes/finger_tip.stl scale=0.001 0.001 0.001; visual mesh filename=package://allegro_hand_description/meshes/finger_tip.stl scale=0.001 0.001 0.001
- link link_12_0: geometry collision mesh filename=package://allegro_hand_description/meshes/t1_set.stl scale=0.001 0.001 0.001; visual mesh filename=package://allegro_hand_description/meshes/t1_set.stl scale=0.001 0.001 0.001
- link link_13_0: geometry collision mesh filename=package://allegro_hand_description/meshes/t2_set.stl scale=0.001 0.001 0.001; visual mesh filename=package://allegro_hand_description/meshes/t2_set.stl scale=0.001 0.001 0.001
- link link_14_0: geometry collision mesh filename=package://allegro_hand_description/meshes/t3_set.stl scale=0.001 0.001 0.001; visual mesh filename=package://allegro_hand_description/meshes/t3_set.stl scale=0.001 0.001 0.001
- link link_15_0: geometry collision mesh filename=package://allegro_hand_description/meshes/t4_set.stl scale=0.001 0.001 0.001; visual mesh filename=package://allegro_hand_description/meshes/t4_set.stl scale=0.001 0.001 0.001
- link link_15_0_tip: geometry collision mesh filename=package://allegro_hand_description/meshes/finger_tip_silico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 scale=0.001 0.001 0.001; visual mesh filename=package://allegro_hand_description/meshes/finger_tip_silico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 scale=0.001 0.001 0.001
- link link_1_0: geometry collision mesh filename=package://allegro_hand_description/meshes/new_l2.stl scale=0.001 0.001 0.001; visual mesh filename=package://allegro_hand_description/meshes/new_l2.stl scale=0.001 0.001 0.001
- link link_2_0: geometry collision mesh filename=package://allegro_hand_description/meshes/new_l3.stl scale=0.001 0.001 0.001; visual mesh filename=package://allegro_hand_description/meshes/new_l3.stl scale=0.001 0.001 0.001
- link link_3_0: geometry collision mesh filename=package://allegro_hand_description/meshes/new_l4.stl scale=0.001 0.001 0.001; visual mesh filename=package://allegro_hand_description/meshes/new_l4.stl scale=0.001 0.001 0.001
- link link_3_0_tip: geometry collision mesh filename=package://allegro_hand_description/meshes/finger_tip.stl scale=0.001 0.001 0.001; visual mesh filename=package://allegro_hand_description/meshes/finger_tip.stl scale=0.001 0.001 0.001
- link link_4_0: geometry collision mesh filename=package://allegro_hand_description/meshes/new_l1.stl scale=0.001 0.001 0.001; visual mesh filename=package://allegro_hand_description/meshes/new_l1.stl scale=0.001 0.001 0.001
- link link_5_0: geometry collision mesh filename=package://allegro_hand_description/meshes/new_l2.stl scale=0.001 0.001 0.001; visual mesh filename=package://allegro_hand_description/meshes/new_l2.stl scale=0.001 0.001 0.001
- link link_6_0: geometry collision mesh filename=package://allegro_hand_description/meshes/new_l3.stl scale=0.001 0.001 0.001; visual mesh filename=package://allegro_hand_description/meshes/new_l3.stl scale=0.001 0.001 0.001
- link link_7_0: geometry collision mesh filename=package://allegro_hand_description/meshes/new_l4.stl scale=0.001 0.001 0.001; visual mesh filename=package://allegro_hand_description/meshes/new_l4.stl scale=0.001 0.001 0.001
- link link_7_0_tip: geometry collision mesh filename=package://allegro_hand_description/meshes/finger_tip.stl scale=0.001 0.001 0.001; visual mesh filename=package://allegro_hand_description/meshes/finger_tip.stl scale=0.001 0.001 0.001
- link link_8_0: geometry collision mesh filename=package://allegro_hand_description/meshes/new_l1.stl scale=0.001 0.001 0.001; visual mesh filename=package://allegro_hand_description/meshes/new_l1.stl scale=0.001 0.001 0.001
- link link_9_0: geometry collision mesh filename=package://allegro_hand_description/meshes/new_l2.stl scale=0.001 0.001 0.001; visual mesh filename=package://allegro_hand_description/meshes/new_l2.stl scale=0.001 0.001 0.001
- link palm_link: geometry collision mesh filename=package://allegro_hand_description/meshes/palm.stl scale=0.001 0.001 0.001; visual mesh filename=package://allegro_hand_description/meshes/palm.stl scale=0.001 0.001 0.001
