Commit message: position and effort hw interfaces

File: src/allegro_hand_description/urdf/allegro_hand_description_left_B.urdf (robot description, URDF)
Before this commit: robot allegro_hand_left, 22 links, 21 joints
Links:
- link link_0_0: mass 0.0176 -> 0.0242; geometry collision mesh filename=package://allegro_hand_description/meshes/new_l1.stl scale=0.001 0.001 0.001; visual mesh filename=package://allegro_hand_description/meshes/new_l1.stl scale=0.001 0.001 0.001
- link link_10_0: mass 0.0367 -> 0.0314; geometry collision mesh filename=package://allegro_hand_description/meshes/new_l3.stl scale=0.001 0.001 0.001; visual mesh filename=package://allegro_hand_description/meshes/new_l3.stl scale=0.001 0.001 0.001
- link link_11_0: mass 0.004 -> 0.0275; geometry collision mesh filename=package://allegro_hand_description/meshes/new_l4.stl scale=0.001 0.001 0.001; visual mesh filename=package://allegro_hand_description/meshes/new_l4.stl scale=0.001 0.001 0.001
- link link_11_0_tip: mass 0.0017 -> 0.0018; geometry collision mesh filename=package://allegro_hand_description/meshes/finger_tip.stl scale=0.001 0.001 0.001; visual mesh filename=package://allegro_hand_description/meshes/finger_tip.stl scale=0.001 0.001 0.001
- link link_12_0: mass 0.0446 -> 0.0416; geometry collision mesh filename=package://allegro_hand_description/meshes/t1_set.stl scale=0.001 0.001 0.001; visual mesh filename=package://allegro_hand_description/meshes/t1_set.stl scale=0.001 0.001 0.001
- link link_13_0: mass 0.0173 -> 0.0224; geometry collision mesh filename=package://allegro_hand_description/meshes/t2_set.stl scale=0.001 0.001 0.001; visual mesh filename=package://allegro_hand_description/meshes/t2_set.stl scale=0.001 0.001 0.001
- link link_14_0: mass 0.03607 -> 0.0315; geometry collision mesh filename=package://allegro_hand_description/meshes/t3_set.stl scale=0.001 0.001 0.001; visual mesh filename=package://allegro_hand_description/meshes/t3_set.stl scale=0.001 0.001 0.001
- link link_15_0: mass 0.0334 -> 0.0545; geometry collision mesh filename=package://allegro_hand_description/meshes/t4_set.stl scale=0.001 0.001 0.001; visual mesh filename=package://allegro_hand_description/meshes/t4_set.stl scale=0.001 0.001 0.001
- link link_15_0_tip: mass 0.0014 -> 0.0015; geometry collision mesh filename=package://allegro_hand_description/meshes/finger_tip_silico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 scale=0.001 0.001 0.001; visual mesh filename=package://allegro_hand_description/meshes/finger_tip_silico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 scale=0.001 0.001 0.001
- link link_1_0: mass 0.086 -> 0.078; geometry collision mesh filename=package://allegro_hand_description/meshes/new_l2.stl scale=0.001 0.001 0.001; visual mesh filename=package://allegro_hand_description/meshes/new_l2.stl scale=0.001 0.001 0.001
- link link_2_0: mass 0.0367 -> 0.0314; geometry collision mesh filename=package://allegro_hand_description/meshes/new_l3.stl scale=0.001 0.001 0.001; visual mesh filename=package://allegro_hand_description/meshes/new_l3.stl scale=0.001 0.001 0.001
- link link_3_0: mass 0.004 -> 0.0275; geometry collision mesh filename=package://allegro_hand_description/meshes/new_l4.stl scale=0.001 0.001 0.001; visual mesh filename=package://allegro_hand_description/meshes/new_l4.stl scale=0.001 0.001 0.001
- link link_3_0_tip: mass 0.0017 -> 0.0018; geometry collision mesh filename=package://allegro_hand_description/meshes/finger_tip.stl scale=0.001 0.001 0.001; visual mesh filename=package://allegro_hand_description/meshes/finger_tip.stl scale=0.001 0.001 0.001
- link link_4_0: mass 0.0176 -> 0.0242; geometry collision mesh filename=package://allegro_hand_description/meshes/new_l1.stl scale=0.001 0.001 0.001; visual mesh filename=package://allegro_hand_description/meshes/new_l1.stl scale=0.001 0.001 0.001
- link link_5_0: mass 0.086 -> 0.078; geometry collision mesh filename=package://allegro_hand_description/meshes/new_l2.stl scale=0.001 0.001 0.001; visual mesh filename=package://allegro_hand_description/meshes/new_l2.stl scale=0.001 0.001 0.001
- link link_6_0: mass 0.0367 -> 0.0314; geometry collision mesh filename=package://allegro_hand_description/meshes/new_l3.stl scale=0.001 0.001 0.001; visual mesh filename=package://allegro_hand_description/meshes/new_l3.stl scale=0.001 0.001 0.001
- link link_7_0: mass 0.004 -> 0.0275; geometry collision mesh filename=package://allegro_hand_description/meshes/new_l4.stl scale=0.001 0.001 0.001; visual mesh filename=package://allegro_hand_description/meshes/new_l4.stl scale=0.001 0.001 0.001
- link link_7_0_tip: mass 0.0017 -> 0.0018; geometry collision mesh filename=package://allegro_hand_description/meshes/finger_tip.stl scale=0.001 0.001 0.001; visual mesh filename=package://allegro_hand_description/meshes/finger_tip.stl scale=0.001 0.001 0.001
- link link_8_0: mass 0.0176 -> 0.0242; geometry collision mesh filename=package://allegro_hand_description/meshes/new_l1.stl scale=0.001 0.001 0.001; visual mesh filename=package://allegro_hand_description/meshes/new_l1.stl scale=0.001 0.001 0.001
- link link_9_0: mass 0.086 -> 0.078; geometry collision mesh filename=package://allegro_hand_description/meshes/new_l2.stl scale=0.001 0.001 0.001; visual mesh filename=package://allegro_hand_description/meshes/new_l2.stl scale=0.001 0.001 0.001
- link palm_link: geometry collision mesh filename=package://allegro_hand_description/meshes/left_hand_G.stl scale=0.001 0.001 0.001; visual mesh filename=package://allegro_hand_description/meshes/left_hand_G.stl scale=0.001 0.001 0.001

File: src/allegro_hand_description/urdf/allegro_hand_description_right_A.urdf (robot description, URDF)
Before this commit: robot allegro_hand_right, 22 links, 21 joints
Links:
- link link_0_0: geometry collision mesh filename=package://allegro_hand_description/meshes/l1.stl scale=0.001 0.001 0.001; visual mesh filename=package://allegro_hand_description/meshes/l1.stl scale=0.001 0.001 0.001
- link link_10_0: geometry collision mesh filename=package://allegro_hand_description/meshes/l3.stl scale=0.001 0.001 0.001; visual mesh filename=package://allegro_hand_description/meshes/l3.stl scale=0.001 0.001 0.001
- link link_11_0: geometry collision mesh filename=package://allegro_hand_description/meshes/l4.stl scale=0.001 0.001 0.001; visual mesh filename=package://allegro_hand_description/meshes/l4.stl scale=0.001 0.001 0.001
- link link_11_0_tip: geometry collision mesh filename=package://allegro_hand_description/meshes/finger_tip.stl scale=0.001 0.001 0.001; visual mesh filename=package://allegro_hand_description/meshes/finger_tip.stl scale=0.001 0.001 0.001
- link link_12_0: geometry collision mesh filename=package://allegro_hand_description/meshes/t1_set.stl scale=0.001 0.001 0.001; visual mesh filename=package://allegro_hand_description/meshes/t1_set.stl scale=0.001 0.001 0.001
- link link_13_0: geometry collision mesh filename=package://allegro_hand_description/meshes/t2_set.stl scale=0.001 0.001 0.001; visual mesh filename=package://allegro_hand_description/meshes/t2_set.stl scale=0.001 0.001 0.001
- link link_14_0: geometry collision mesh filename=package://allegro_hand_description/meshes/t3_set.stl scale=0.001 0.001 0.001; visual mesh filename=package://allegro_hand_description/meshes/t3_set.stl scale=0.001 0.001 0.001
- link link_15_0: geometry collision mesh filename=package://allegro_hand_description/meshes/t4_set.stl scale=0.001 0.001 0.001; visual mesh filename=package://allegro_hand_description/meshes/t4_set.stl scale=0.001 0.001 0.001
- link link_15_0_tip: geometry collision mesh filename=package://allegro_hand_description/meshes/finger_tip_silico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 scale=0.001 0.001 0.001; visual mesh filename=package://allegro_hand_description/meshes/finger_tip_silico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 scale=0.001 0.001 0.001
- link link_1_0: geometry collision mesh filename=package://allegro_hand_description/meshes/l2.stl scale=0.001 0.001 0.001; visual mesh filename=package://allegro_hand_description/meshes/l2.stl scale=0.001 0.001 0.001
- link link_2_0: geometry collision mesh filename=package://allegro_hand_description/meshes/l3.stl scale=0.001 0.001 0.001; visual mesh filename=package://allegro_hand_description/meshes/l3.stl scale=0.001 0.001 0.001
- link link_3_0: geometry collision mesh filename=package://allegro_hand_description/meshes/l4.stl scale=0.001 0.001 0.001; visual mesh filename=package://allegro_hand_description/meshes/l4.stl scale=0.001 0.001 0.001
- link link_3_0_tip: geometry collision mesh filename=package://allegro_hand_description/meshes/finger_tip.stl scale=0.001 0.001 0.001; visual mesh filename=package://allegro_hand_description/meshes/finger_tip.stl scale=0.001 0.001 0.001
- link link_4_0: geometry collision mesh filename=package://allegro_hand_description/meshes/l1.stl scale=0.001 0.001 0.001; visual mesh filename=package://allegro_hand_description/meshes/l1.stl scale=0.001 0.001 0.001
- link link_5_0: geometry collision mesh filename=package://allegro_hand_description/meshes/l2.stl scale=0.001 0.001 0.001; visual mesh filename=package://allegro_hand_description/meshes/l2.stl scale=0.001 0.001 0.001
- link link_6_0: geometry collision mesh filename=package://allegro_hand_description/meshes/l3.stl scale=0.001 0.001 0.001; visual mesh filename=package://allegro_hand_description/meshes/l3.stl scale=0.001 0.001 0.001
- link link_7_0: geometry collision mesh filename=package://allegro_hand_description/meshes/l4.stl scale=0.001 0.001 0.001; visual mesh filename=package://allegro_hand_description/meshes/l4.stl scale=0.001 0.001 0.001
- link link_7_0_tip: geometry collision mesh filename=package://allegro_hand_description/meshes/finger_tip.stl scale=0.001 0.001 0.001; visual mesh filename=package://allegro_hand_description/meshes/finger_tip.stl scale=0.001 0.001 0.001
- link link_8_0: geometry collision mesh filename=package://allegro_hand_description/meshes/l1.stl scale=0.001 0.001 0.001; visual mesh filename=package://allegro_hand_description/meshes/l1.stl scale=0.001 0.001 0.001
- link link_9_0: geometry collision mesh filename=package://allegro_hand_description/meshes/l2.stl scale=0.001 0.001 0.001; visual mesh filename=package://allegro_hand_description/meshes/l2.stl scale=0.001 0.001 0.001
- link palm_link: geometry collision mesh filename=package://allegro_hand_description/meshes/palm.stl scale=0.001 0.001 0.001; visual mesh filename=package://allegro_hand_description/meshes/palm.stl scale=0.001 0.001 0.001

File: src/allegro_hand_description/urdf/allegro_hand_description_right_B.urdf (robot description, URDF)
Before this commit: robot allegro_hand_right, 22 links, 21 joints
Links:
- added link wrist
- link link_0_0: mass 0.0176 -> 0.0242
- link link_10_0: mass 0.0367 -> 0.0314
- link link_11_0: mass 0.004 -> 0.0275; geometry collision mesh filename=package://allegro_hand_description/meshes/ft_fingertip_v2.s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 scale=0.001 0.001 0.001; visual mesh filename=package://allegro_hand_description/meshes/ft_fingertip_v2.s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 scale=0.001 0.001 0.001
- link link_11_0_tip: mass 0.0017 -> None; geometry 
- link link_12_0: mass 0.0446 -> 0.0416
- link link_13_0: mass 0.0173 -> 0.0224
- link link_14_0: mass 0.03607 -> 0.0315
- link link_15_0: mass 0.0334 -> 0.0545; geometry collision mesh filename=package://allegro_hand_description/meshes/ft_thumbtip_v2.stl scale=0.001 0.001 0.001; visual mesh filename=package://allegro_hand_description/meshes/ft_thumbtip_v2.stl scale=0.001 0.001 0.001
- link link_15_0_tip: mass 0.0014 -> None; geometry 
- link link_1_0: mass 0.086 -> 0.078
- link link_2_0: mass 0.0367 -> 0.0314
- link link_3_0: mass 0.004 -> 0.0275; geometry collision mesh filename=package://allegro_hand_description/meshes/ft_fingertip_v2.s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 scale=0.001 0.001 0.001; visual mesh filename=package://allegro_hand_description/meshes/ft_fingertip_v2.s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 scale=0.001 0.001 0.001
- link link_3_0_tip: mass 0.0017 -> None; geometry 
- link link_4_0: mass 0.0176 -> 0.0242
- link link_5_0: mass 0.086 -> 0.078
- link link_6_0: mass 0.0367 -> 0.0314
- link link_7_0: mass 0.004 -> 0.0275; geometry collision mesh filename=package://allegro_hand_description/meshes/ft_fingertip_v2.s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 scale=0.001 0.001 0.001; visual mesh filename=package://allegro_hand_description/meshes/ft_fingertip_v2.s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 scale=0.001 0.001 0.001
- link link_7_0_tip: mass 0.0017 -> None; geometry 
- link link_8_0: mass 0.0176 -> 0.0242
- link link_9_0: mass 0.086 -> 0.078
Joints:
- added joint wrist_joint: type fixed, parent palm_link, child wrist, origin xyz=0 0 -0.1005 rpy=0 0 0
- joint joint_11_0_tip: origin xyz=0 0 0.04 rpy=0 0 0 -> xyz=0.008 0 0.04 rpy=1.57 0.0 1.57
- joint joint_15_0_tip: origin xyz=0 0 0.05 rpy=0 0 0 -> xyz=0.008 0 0.05 rpy=1.57 0.0 1.57
- joint joint_3_0_tip: origin xyz=0 0 0.04 rpy=0 0 0 -> xyz=0.008 0 0.04 rpy=1.57 0.0 1.57
- joint joint_7_0_tip: origin xyz=0 0 0.04 rpy=0 0 0 -> xyz=0.008 0 0.04 rpy=1.57 0.0 1.57

File: src/allegro_hand_moveit/config/allegro_hand_right_B.urdf.xacro (robot description, xacro)
@@ -2,8 +2,13 @@
 <robot xmlns:xacro="http://www.ros.org/wiki/xacro" name="allegro_hand">
     <xacro:arg name="initial_positions_file" default="initial_positions.yaml" />
+    <!-- <xacro:include filename="$(find allegro_hand_moveit)/config/allegro_hand_ros2control.xacro" /> -->
     <!-- Import allegro_hand urdf file -->
-    <xacro:include filename="$(find allegro_hand_controllers)/urdf/allegro_hand_description_right_B.urdf" />
+    <!-- <xacro:include filename="$(find allegro_hand_controllers)/urdf/allegro_hand_description_right_B.urdf" /> -->
     <!-- Import control_xacro -->
-    <xacro:include filename="allegro_hand.ros2_control.xacro" />
-    <xacro:allegro_hand_ros2_control name="FakeSystem" initial_positions_file="$(arg initial_positions_file)"/>
+    <!-- <xacro:include filename="allegro_hand.ros2_control.xacro" /> -->
+    <!-- <xacro:allegro_hand_ros2_control name="FakeSystem" initial_positions_file="$(arg initial_positions_file)"/> -->
+    <!-- LEO (LOAD custom controllers defined in bringup)-->
+    <!-- <xacro:arg name="ros2_control_hardware_type" default="physical_device" /> -->
+    <!-- <xacro:arg name="ros2_control_hardware_type" default="mock_components" /> -->
+    <xacro:include filename="$(find allegro_hand_bringup)/config/allegro_hand_ros2control.xacro" />
 </robot>
